File: hardware/schema/schema.sch (KiCad schematic (older format))
At the start: 5 parts

Commit message: Core bugfixes + Hardware design
Parts:
- removed U?: BME280MOD, symbol bme280mod:BME280MOD
- added C1: 47u, w_capacitors:CP_5x11mm_hor, symbol Device:CP
- added J2: Conn_01x04, Connector_PinHeader_2.54mm:PinHeader_1x04_P2.54mm_Vertical, symbol Connector_Generic:Conn_01x04
- J1: renamed from J?; footprint (none) -> Battery:BatteryHolder_Keystone_107_1x23mm
- R1, R2: renamed from R?; footprint (none) -> Resistor_THT:R_Axial_DIN0204_L3.6mm_D1.6mm_P7.62mm_Horizontal
- U1: renamed from U?; footprint (none) -> moteino:moteino-r6; symbol moteino:MoteinoR6 -> moteino:MoteinoR6_1
Connections:
- net +3V0: now also U1.15 (3.3V), U1.27 (3.3V), C1.1, J2.1 (Pin_1); no longer U1.~ (VIN)
- net Batt: now also U1.17 (A0); no longer U1.~ (VIN)
- net GND: now also U1.16 (GND), U1.29 (GND), C1.2, J2.2 (Pin_2)
- net SCL: now also U1.22 (A5(SCL)), J2.3 (Pin_3); no longer U1.~ (VIN)
- net SDA: now also U1.21 (A4(SDA)), J2.4 (Pin_4); no longer U1.~ (VIN)
Other:
- note added: "CR2450 Holder"
- note added: "Power Booster"
- note removed: "CR2560 Holder"
Changed lines of the file:
@@
 $EndDescr
 $Comp
-L moteino:MoteinoR6 U?
+L moteino:MoteinoR6_1 U1
 U 1 1 6185BA0B
 P 4400 3500
-F 0 "U?" H 4400 2411 50  0000 C CNN
-F 1 "MoteinoR6" H 4400 2320 50  0000 C CNN
-F 2 "" H 4150 3350 50  0001 C CNN
+F 0 "U1" H 4750 2450 50  0000 C CNN
+F 1 "MoteinoR6" H 4100 2450 50  0000 C CNN
+F 2 "moteino:moteino-r6" H 4150 3350 50  0001 C CNN
 F 3 "" H 4150 3350 50  0001 C CNN
 	1    4400 3500
@@
 $EndComp
 $Comp
-L bme280mod:BME280MOD U?
-U 1 1 6185C261
-P 6750 2950
-F 0 "U?" H 6522 2996 50  0000 R CNN
-F 1 "BME280MOD" H 6522 2905 50  0000 R CNN
-F 2 "" H 6700 3050 50  0001 C CNN
-F 3 "" H 6700 3050 50  0001 C CNN
-	1    6750 2950
-	-1   0    0    -1
-$EndComp
-$Comp
-L Connector_Generic:Conn_01x02 J?
+L Connector_Generic:Conn_01x02 J1
 U 1 1 6185DB0E
 P 5650 4350
-F 0 "J?" H 5730 4342 50  0000 L CNN
+F 0 "J1" H 5730 4342 50  0000 L CNN
 F 1 "CR2450 Battery Holder" H 5730 4251 50  0000 L CNN
-F 2 "" H 5650 4350 50  0001 C CNN
+F 2 "Battery:BatteryHolder_Keystone_107_1x23mm" H 5650 4350 50  0001 C CNN
 F 3 "~" H 5650 4350 50  0001 C CNN
 	1    5650 4350
@@
 $EndComp
 $Comp
-L Device:R R?
+L Device:R R1
 U 1 1 6185E322
 P 5600 2800
-F 0 "R?" H 5670 2846 50  0000 L CNN
+F 0 "R1" H 5670 2846 50  0000 L CNN
 F 1 "680k" H 5670 2755 50  0000 L CNN
-F 2 "" V 5530 2800 50  0001 C CNN
+F 2 "Resistor_THT:R_Axial_DIN0204_L3.6mm_D1.6mm_P7.62mm_Horizontal" V 5530 2800 50  0001 C CNN
 F 3 "~" H 5600 2800 50  0001 C CNN
 	1    5600 2800
@@
 $EndComp
 $Comp
-L Device:R R?
+L Device:R R2
 U 1 1 6185E5F7
 P 5600 3300
-F 0 "R?" H 5670 3346 50  0000 L CNN
+F 0 "R2" H 5670 3346 50  0000 L CNN
 F 1 "330" H 5670 3255 50  0000 L CNN
-F 2 "" V 5530 3300 50  0001 C CNN
+F 2 "Resistor_THT:R_Axial_DIN0204_L3.6mm_D1.6mm_P7.62mm_Horizontal" V 5530 3300 50  0001 C CNN
 F 3 "~" H 5600 3300 50  0001 C CNN
 	1    5600 3300
@@
 	5600 3050 5600 3150
 $Comp
-L power:+3V0 #PWR?
+L power:+3V0 #PWR01
 U 1 1 61860534
-P 4450 2350
-F 0 "#PWR?" H 4450 2200 50  0001 C CNN
-F 1 "+3V0" H 4465 2523 50  0000 C CNN
-F 2 "" H 4450 2350 50  0001 C CNN
-F 3 "" H 4450 2350 50  0001 C CNN
-	1    4450 2350
-	1    0    0    -1
-$EndComp
-$Comp
-L power:+3V0 #PWR?
+P 4300 2350
+F 0 "#PWR01" H 4300 2200 50  0001 C CNN
+F 1 "+3V0" H 4315 2523 50  0000 C CNN
+F 2 "" H 4300 2350 50  0001 C CNN
+F 3 "" H 4300 2350 50  0001 C CNN
+	1    4300 2350
+	1    0    0    -1
+$EndComp
+$Comp
+L power:+3V0 #PWR09
 U 1 1 618608EC
-P 6350 2700
-F 0 "#PWR?" H 6350 2550 50  0001 C CNN
-F 1 "+3V0" H 6365 2873 50  0000 C CNN
-F 2 "" H 6350 2700 50  0001 C CNN
-F 3 "" H 6350 2700 50  0001 C CNN
-	1    6350 2700
-	1    0    0    -1
-$EndComp
-$Comp
-L power:+3V0 #PWR?
+P 7100 3300
+F 0 "#PWR09" H 7100 3150 50  0001 C CNN
+F 1 "+3V0" H 7115 3473 50  0000 C CNN
+F 2 "" H 7100 3300 50  0001 C CNN
+F 3 "" H 7100 3300 50  0001 C CNN
+	1    7100 3300
+	1    0    0    -1
+$EndComp
+$Comp
+L power:+3V0 #PWR02
 U 1 1 61860DF0
 P 5350 4250
-F 0 "#PWR?" H 5350 4100 50  0001 C CNN
+F 0 "#PWR02" H 5350 4100 50  0001 C CNN
 F 1 "+3V0" H 5365 4423 50  0000 C CNN
 F 2 "" H 5350 4250 50  0001 C CNN
@@
 $EndComp
 $Comp
-L power:GND #PWR?
+L power:GND #PWR05
 U 1 1 618612A2
 P 5600 3600
-F 0 "#PWR?" H 5600 3350 50  0001 C CNN
+F 0 "#PWR05" H 5600 3350 50  0001 C CNN
 F 1 "GND" H 5605 3427 50  0000 C CNN
 F 2 "" H 5600 3600 50  0001 C CNN
@@
 $EndComp
 $Comp
-L power:GND #PWR?
+L power:GND #PWR08
 U 1 1 6186150D
-P 6300 2900
-F 0 "#PWR?" H 6300 2650 50  0001 C CNN
-F 1 "GND" V 6305 2772 50  0000 R CNN
-F 2 "" H 6300 2900 50  0001 C CNN
-F 3 "" H 6300 2900 50  0001 C CNN
-	1    6300 2900
+P 7050 3500
+F 0 "#PWR08" H 7050 3250 50  0001 C CNN
+F 1 "GND" V 7055 3372 50  0000 R CNN
+F 2 "" H 7050 3500 50  0001 C CNN
+F 3 "" H 7050 3500 50  0001 C CNN
+	1    7050 3500
 	0    1    1    0
 $EndComp
@@
 Text GLabel 3750 3800 0    50   Input ~ 0
 SCL
-Text GLabel 6300 3000 0    50   Input ~ 0
+Text GLabel 7050 3700 0    50   Input ~ 0
 SDA
-Text GLabel 6300 3100 0    50   Input ~ 0
+Text GLabel 7050 3600 0    50   Input ~ 0
 SCL
 Wire Wire Line
@@
 	5350 4350 5350 4250
 $Comp
-L power:GND #PWR?
+L power:GND #PWR03
 U 1 1 61862A91
 P 5350 4550
-F 0 "#PWR?" H 5350 4300 50  0001 C CNN
+F 0 "#PWR03" H 5350 4300 50  0001 C CNN
 F 1 "GND" H 5355 4377 50  0000 C CNN
 F 2 "" H 5350 4550 50  0001 C CNN
@@
 	5600 3450 5600 3600
 Wire Wire Line
-	6450 2800 6350 2800
-Wire Wire Line
-	6350 2800 6350 2700
-Wire Wire Line
-	6450 2900 6300 2900
-Wire Wire Line
-	6450 3000 6300 3000
-Wire Wire Line
-	6450 3100 6300 3100
-Wire Wire Line
-	4450 2350 4450 2500
+	7200 3400 7100 3400
+Wire Wire Line
+	7100 3400 7100 3300
+Wire Wire Line
+	7200 3500 7050 3500
+Wire Wire Line
+	7200 3600 7050 3600
+Wire Wire Line
+	7200 3700 7050 3700
 Wire Wire Line
 	3900 3300 3750 3300
@@
 NoConn ~ 4900 4050
 NoConn ~ 4900 4150
-NoConn ~ 3900 2950
-NoConn ~ 3900 3050
-NoConn ~ 3900 3150
 NoConn ~ 3900 3400
 NoConn ~ 3900 3500
@@
 	6700 3900 5150 3900
 Wire Notes Line
-	6000 2350 6000 3250
-Wire Notes Line
-	6000 3250 7500 3250
-Wire Notes Line
-	7500 3250 7500 2350
-Wire Notes Line
-	7500 2350 6000 2350
+	6750 2950 6750 3850
+Wire Notes Line
+	6750 3850 8250 3850
+Wire Notes Line
+	8250 3850 8250 2950
+Wire Notes Line
+	8250 2950 6750 2950
 Text Notes 3450 2100 0    50   ~ 0
 Moteino R6 with RFM69HCW
 Text Notes 5200 2200 0    50   ~ 0
 Battery Level \nMeasure
-Text Notes 6050 2450 0    50   ~ 0
+Text Notes 6800 3050 0    50   ~ 0
 BME280 Module
-Text Notes 6100 4050 0    50   ~ 0
-CR2560 Holder
+Text Notes 5700 4000 0    50   ~ 0
+CR2450 Holder
 NoConn ~ 3900 2850
 $Comp
-L power:+3V0 #PWR?
+L power:+3V0 #PWR04
 U 1 1 61889CE5
 P 5600 2400
-F 0 "#PWR?" H 5600 2250 50  0001 C CNN
+F 0 "#PWR04" H 5600 2250 50  0001 C CNN
 F 1 "+3V0" H 5615 2573 50  0000 C CNN
 F 2 "" H 5600 2400 50  0001 C CNN
@@
 	1    0    0    -1
 $EndComp
+$Comp
+L Device:CP C1
+U 1 1 61894DB0
+P 6300 3250
+F 0 "C1" H 6418 3296 50  0000 L CNN
+F 1 "47u" H 6418 3205 50  0000 L CNN
+F 2 "w_capacitors:CP_5x11mm_hor" H 6338 3100 50  0001 C CNN
+F 3 "~" H 6300 3250 50  0001 C CNN
+	1    6300 3250
+	1    0    0    -1
+$EndComp
+$Comp
+L power:+3V0 #PWR06
+U 1 1 61895242
+P 6300 2950
+F 0 "#PWR06" H 6300 2800 50  0001 C CNN
+F 1 "+3V0" H 6315 3123 50  0000 C CNN
+F 2 "" H 6300 2950 50  0001 C CNN
+F 3 "" H 6300 2950 50  0001 C CNN
+	1    6300 2950
+	1    0    0    -1
+$EndComp
+$Comp
+L power:GND #PWR07
+U 1 1 61895545
+P 6300 3600
+F 0 "#PWR07" H 6300 3350 50  0001 C CNN
+F 1 "GND" H 6305 3427 50  0000 C CNN
+F 2 "" H 6300 3600 50  0001 C CNN
+F 3 "" H 6300 3600 50  0001 C CNN
+	1    6300 3600
+	1    0    0    -1
+$EndComp
+Wire Wire Line
+	6300 3100 6300 2950
+Wire Wire Line
+	6300 3400 6300 3600
+Wire Notes Line
+	6000 2600 6000 3850
+Wire Notes Line
+	6000 3850 6700 3850
+Wire Notes Line
+	6700 3850 6700 2600
+Wire Notes Line
+	6700 2600 6000 2600
+Text Notes 6050 2700 0    50   ~ 0
+Power Booster
+NoConn ~ 3900 4100
+NoConn ~ 3900 4200
+$Comp
+L Connector_Generic:Conn_01x04 J2
+U 1 1 618AD8FF
+P 7400 3500
+F 0 "J2" H 7480 3492 50  0000 L CNN
+F 1 "Conn_01x04" H 7480 3401 50  0000 L CNN
+F 2 "Connector_PinHeader_2.54mm:PinHeader_1x04_P2.54mm_Vertical" H 7400 3500 50  0001 C CNN
+F 3 "~" H 7400 3500 50  0001 C CNN
+	1    7400 3500
+	1    0    0    -1
+$EndComp
+$Comp
+L power:GND #PWR0101
+U 1 1 618B077A
+P 4400 4600
+F 0 "#PWR0101" H 4400 4350 50  0001 C CNN
+F 1 "GND" H 4405 4427 50  0000 C CNN
+F 2 "" H 4400 4600 50  0001 C CNN
+F 3 "" H 4400 4600 50  0001 C CNN
+	1    4400 4600
+	1    0    0    -1
+$EndComp
+Wire Wire Line
+	4400 4600 4400 4500
+Wire Wire Line
+	3700 2950 3700 2850
+Wire Wire Line
+	3900 2950 3700 2950
+Wire Wire Line
+	3900 3050 3700 3050
+$Comp
+L power:GND #PWR0103
+U 1 1 618CE45E
+P 3700 3050
+F 0 "#PWR0103" H 3700 2800 50  0001 C CNN
+F 1 "GND" H 3705 2877 50  0000 C CNN
+F 2 "" H 3700 3050 50  0001 C CNN
+F 3 "" H 3700 3050 50  0001 C CNN
+	1    3700 3050
+	0    1    1    0
+$EndComp
+$Comp
+L power:+3V0 #PWR0102
+U 1 1 618CDF1B
+P 3700 2850
+F 0 "#PWR0102" H 3700 2700 50  0001 C CNN
+F 1 "+3V0" H 3715 3023 50  0000 C CNN
+F 2 "" H 3700 2850 50  0001 C CNN
+F 3 "" H 3700 2850 50  0001 C CNN
+	1    3700 2850
+	1    0    0    -1
+$EndComp
+Wire Wire Line
+	4300 2500 4300 2350
+NoConn ~ 4450 2500
 $EndSCHEMATC
